Commit message: updated ros2_control.xacro (removed Gazebo, put in for real robot), but need a real encoder (won't work atm when controlling driving)

File: description/ros2_control.xacro (robot description, xacro)
@@ -1,7 +1,38 @@
 <?xml version="1.0"?>
 <robot xmlns:xacro="http://www.ros.org/wiki/xacro">
+<!--
     <ros2_control name="GazeboSystem" type="system">
         <hardware>
             <plugin>gazebo_ros2_control/GazeboSystem</plugin>
+        </hardware>
+        <joint name="left_wheel_joint">
+            <command_interface name="velocity">
+                <param name="min">-10</param>
+                <param name="max">10</param>
+            </command_interface>
+            <state_interface name="velocity"/>
+            <state_interface name="position"/>
+        </joint>
+        <joint name="right_wheel_joint">
+            <command_interface name="velocity">
+                <param name="min">-10</param>
+                <param name="max">10</param>
+            </command_interface>
+            <state_interface name="velocity"/>
+            <state_interface name="position"/>
+        </joint>
+    </ros2_control> -->
+     <ros2_control name="RealRobot" type="system">
+        <hardware>
+            <!-- TEST Values for plugin below are from Josh (tutorial) and not from our motors
+            Our motors don't have an encoder, unable to get the motor's specific parameter values atm -->
+            <plugin>diffdrive_arduino/DiffDriveArduino</plugin>
+            <param name="left_wheel_name">left_wheel_joint</param>
+            <param name="right_wheel_name">right_wheel_joint</param>
+            <param name="loop_rate">30</param>
+            <param name="device">/dev/ttyUSB0</param>
+            <param name="baud_rate">57600</param>
+            <param name="timeout">1000</param>
+            <param name="enc_counts_per_rev">1</param> <!-- TEST Put encoder counts as 1 -->
         </hardware>
         <joint name="left_wheel_joint">
