Commit message: adjust tuning and follow_ball parameters, also updated the core.xacro and controllers.yaml file

File: description/robot_core.xacro (robot description, xacro)
@@ -2,10 +2,10 @@
 <robot xmlns:xacro="http://www.ros.org/wiki/xacro" >
     <xacro:include filename="inertial_macros.xacro"/>
-    <xacro:property name="chassis_length" value="0.335"/>
-    <xacro:property name="chassis_width" value="0.265"/>
-    <xacro:property name="chassis_height" value="0.138"/>
-    <xacro:property name="chassis_mass" value="1.0"/>
-    <xacro:property name="wheel_radius" value="0.034"/>
-    <xacro:property name="wheel_thickness" value="0.026"/>
+    <xacro:property name="chassis_length" value="0.685"/>
+    <xacro:property name="chassis_width" value="0.42"/>
+    <xacro:property name="chassis_height" value="0.23"/>
+    <xacro:property name="chassis_mass" value="1.5"/>
+    <xacro:property name="wheel_radius" value="0.07"/>
+    <xacro:property name="wheel_thickness" value="0.033"/>
     <xacro:property name="wheel_mass" value="0.05"/>
     <xacro:property name="wheel_offset_x" value="0.226"/>

Commit message: (for testing) copied over the my_controllers and robot_core from articubot repo

File: description/robot_core.xacro (robot description, xacro)
@@ -2,10 +2,10 @@
 <robot xmlns:xacro="http://www.ros.org/wiki/xacro" >
     <xacro:include filename="inertial_macros.xacro"/>
-    <xacro:property name="chassis_length" value="0.685"/>
-    <xacro:property name="chassis_width" value="0.42"/>
-    <xacro:property name="chassis_height" value="0.23"/>
-    <xacro:property name="chassis_mass" value="1.5"/>
-    <xacro:property name="wheel_radius" value="0.07"/>
-    <xacro:property name="wheel_thickness" value="0.033"/>
+    <xacro:property name="chassis_length" value="0.335"/>
+    <xacro:property name="chassis_width" value="0.265"/>
+    <xacro:property name="chassis_height" value="0.138"/>
+    <xacro:property name="chassis_mass" value="1.0"/>
+    <xacro:property name="wheel_radius" value="0.033"/>
+    <xacro:property name="wheel_thickness" value="0.026"/>
     <xacro:property name="wheel_mass" value="0.05"/>
     <xacro:property name="wheel_offset_x" value="0.226"/>
