Commit message: made some changes to wheel separation, wheel radius and wheel y offsest

File: install/my_bot/share/my_bot/description/gazebo_control.xacro (robot description, xacro)
@@ -6,9 +6,6 @@
             <left_joint>left_wheel_joint</left_joint>
             <right_joint>right_wheel_joint</right_joint>
-            <!--WHEEL SEPARATION ORIGINALLY 0.35-->
-            <!--NOTE: THESE VALUES ACTUALLY DON'T LINE UP WITH my_controllers.yaml, but might not matter as this is for Gazebo-->
-            <wheel_separation>0.297</wheel_separation>
-            <!--WHEEL DIAMETER ORIGINALLY 0.1-->
-            <wheel_diameter>0.066</wheel_diameter>
+            <wheel_separation>0.35</wheel_separation>
+            <wheel_diameter>0.1</wheel_diameter>
             <!-- Limits -->
             <max_wheel_torque>200</max_wheel_torque>

File: install/my_bot/share/my_bot/description/robot_core.xacro (robot description, xacro)
@@ -6,11 +6,9 @@
     <xacro:property name="chassis_height" value="0.138"/>
     <xacro:property name="chassis_mass" value="1.0"/>
-    <!--WHEEL RADIUS ORIGNALLY = 0.075, 0.037 (articubot_one)-->
-    <xacro:property name="wheel_radius" value="0.072"/>
+    <xacro:property name="wheel_radius" value="0.033"/>
     <xacro:property name="wheel_thickness" value="0.026"/>
     <xacro:property name="wheel_mass" value="0.05"/>
     <xacro:property name="wheel_offset_x" value="0.226"/>
-    <!--WHEEL OFFSET Y ORIGINALLY 0.166-->
-    <xacro:property name="wheel_offset_y" value="0.1485"/>
+    <xacro:property name="wheel_offset_y" value="0.166"/>
     <xacro:property name="wheel_offset_z" value="0.01"/>
     <xacro:property name="caster_wheel_radius" value="0.01"/>
